File: pcb-lite/launch-lite.kicad_sch (KiCad schematic)
At the start: 209 parts, among them J0 TYPE-C-31-M-12, J1 DNP, J6 DNP, U0 USBLC6-2SC6, U1 AT90USB646-MUR, Y0 ECS-160-18-23G-JGN-TR

Commit message: prepare v0
Parts:
- removed C0, C1, C2, C3, C4, C7: 1 uF, launch:C_0402_1005Metric, symbol Device:C
- removed C5, C6: 22pF, Capacitor_SMD:C_0402_1005Metric, symbol Device:C
- removed D19, D20, D26: BAV70,215, Package_TO_SOT_SMD:SOT-23, symbol Device:D_Dual_CommonCathode_AAK
- removed FID3, FID4: Fiducial, Fiducial:Fiducial_0.75mm_Mask1.5mm, symbol Mechanical:Fiducial
- removed H7, H8: MountingHole_Pad, launch:MountingHole, symbol Mechanical:MountingHole_Pad
- removed J0: TYPE-C-31-M-12, Connector_USB:USB_C_Receptacle_HRO_TYPE-C-31-M-12, symbol Connector:USB_C_Receptacle_USB2.0
- removed J1: DNP, Connector:Tag-Connect_TC2030-IDC-FP_2x03_P1.27mm_Vertical, symbol Connector:AVR-ISP-6
- removed J6: DNP, Connector_PinHeader_2.54mm:PinHeader_1x02_P2.54mm_Vertical, symbol Connector_Generic:Conn_01x02
- removed LA1, LA2, LA3, LA4, LA5, LB1, LB2, LB3, LB4, LB5, LC1, LC2, LC3, LC4, LC5, LD1, LD2, LD3, LD4, LD5, LE1, LE2, LE3, LE4, LE5, LF1, LF2, LF3, LF4, LG1, LG2, LG3, LG4, LG5, LH1, LH2, LH3, LH4, LH5, LI1, LI2, LI3, LI4, LI5, LJ1, LJ2, LJ3, LJ4, LJ5, LK1, LK2, LK3, LK4, LK5, LL1, LL2, LL3, LL4, LL5, LM1, LM2, LM3, LM4, LM5, LN1, LN2, LO0, LO1, LO2, LO3: SK6805-EC15, launch:LED_SK6805-EC15, symbol launch:SK6805-EC15
- removed R1, R5: 5.1 k, launch:R_0402_1005Metric, symbol Device:R
- removed R2, R3: 22, launch:R_0402_1005Metric, symbol Device:R
- removed R27: 499, launch:R_0402_1005Metric, symbol Device:R
- removed R4: 10 k, launch:R_0402_1005Metric, symbol Device:R
- removed SWF5, SWK5, SWL5, SWM4, SWM5, SWN3, SWN4, SWN5: CPG151101S11, Kailh:Kailh_socket_MX, symbol Switch:SW_Push
- removed U0: USBLC6-2SC6, Package_TO_SOT_SMD:SOT-23-6, symbol Power_Protection:USBLC6-2SC6
- removed U1: AT90USB646-MUR, Package_DFN_QFN:QFN-64-1EP_9x9mm_P0.5mm_EP7.5x7.5mm, symbol MCU_Microchip_AVR:AT90USB646-M
- removed Y0: ECS-160-18-23G-JGN-TR, Crystal:Crystal_SMD_0603-2Pin_6.0x3.5mm, symbol Device:Crystal
- added J1: Micro_SD_Card_Det1, Connector_Card:microSD_HC_Wuerth_693072010801, symbol Connector:Micro_SD_Card_Det1
- added J2: Conn_02x08_Counter_Clockwise, Connector_PinHeader_2.54mm:PinHeader_2x08_P2.54mm_Vertical_SMD, symbol Connector_Generic:Conn_02x08_Counter_Clockwise
- added J3, J4: Conn_02x20_Counter_Clockwise, symbol Connector_Generic:Conn_02x20_Odd_Even
- added JP1: Jumper_2_Open, Jumper:SolderJumper-2_P1.3mm_Open_Pad1.0x1.5mm, symbol Jumper:Jumper_2_Open
- added U1: CY15B104QN, Package_SO:SOIC-8_3.9x4.9mm_P1.27mm, symbol Memory_NVRAM:FM24C64C
- added U2: Pico, RPi_Pico:RPi_Pico_SMD_TH, symbol MCU_RaspberryPi_and_Boards:Pico
Connections:
- net COLA: now also U2.11 (GPIO8)
- net COLB: now also U2.12 (GPIO9)
- net COLC: now also U2.14 (GPIO10)
- net COLD: now also U2.15 (GPIO11)
- net COLE: now also U2.16 (GPIO12)
- net COLF: now also U2.17 (GPIO13)
- net COLG: now also U2.19 (GPIO14)
- net COLH: now also U2.20 (GPIO15)
- net COLI: now also U2.21 (GPIO16)
- net COLJ: now also U2.22 (GPIO17)
- net COLK: now also U2.24 (GPIO18)
- net COLL: now also U2.25 (GPIO19)
- net COLM: now also U2.26 (GPIO20)
- net COLN: now also U2.27 (GPIO21)
- net GND: now also J1.6 (VSS), J2.10 (Pin_10), J2.7 (Pin_7), J3.15 (Pin_15), J3.16 (Pin_16), J3.25 (Pin_25), J3.26 (Pin_26), J3.35 (Pin_35), J3.36 (Pin_36), J3.5 (Pin_5), J3.6 (Pin_6), J4.15 (Pin_15), J4.16 (Pin_16), J4.25 (Pin_25), J4.26 (Pin_26), J4.35 (Pin_35), J4.36 (Pin_36), J4.5 (Pin_5), J4.6 (Pin_6), U1.4 (VSS), U2.13 (GND), U2.18 (GND), U2.23 (GND), U2.28 (GND), U2.3 (GND), U2.33 (AGND), U2.38 (GND), U2.8 (GND)
- net ROW1: now also U2.5 (GPIO3)
- net ROW2: now also U2.31 (GPIO26_ADC0)
- net ROW3: now also U2.29 (GPIO22)
- net ROW4: now also U2.9 (GPIO6)
- net ROW5: now also U2.10 (GPIO7)
- net VBUS: now also J2.9 (Pin_9), J4.1 (Pin_1), J4.2 (Pin_2), U2.40 (VBUS)
- new net: J1.9 (DET), JP1.2 (B)
- new net: J4.10 (Pin_10), J4.9 (Pin_9)
- new net: J4.11 (Pin_11), J4.12 (Pin_12)
- new net: J4.13 (Pin_13), J4.14 (Pin_14)
- new net: J4.17 (Pin_17), J4.18 (Pin_18)
- new net: J4.19 (Pin_19), J4.20 (Pin_20)
- new net: J4.21 (Pin_21), J4.22 (Pin_22)
- new net: J4.23 (Pin_23), J4.24 (Pin_24)
- new net: J4.27 (Pin_27), J4.28 (Pin_28)
- new net: J4.7 (Pin_7), J4.8 (Pin_8)
- new net: J3.17 (Pin_17), J3.18 (Pin_18)
- new net: J3.19 (Pin_19), J3.20 (Pin_20)
- new net +3.3V: J1.4 (VDD), J2.8 (Pin_8), J4.3 (Pin_3), J4.4 (Pin_4), U1.3 (WP), U1.8 (VDD), U2.39 (VSYS)
- new net EPD_BUSY: J2.1 (Pin_1), J2.16 (Pin_16), J3.27 (Pin_27), J3.28 (Pin_28)
- new net EPD_CLK: J2.13 (Pin_13), J2.5 (Pin_5), J3.37 (Pin_37), J3.38 (Pin_38)
- new net EPD_CS: J2.14 (Pin_14), J2.4 (Pin_4), J3.33 (Pin_33), J3.34 (Pin_34)
- new net EPD_DC/DOUT: J2.11 (Pin_11), J2.3 (Pin_3), J3.31 (Pin_31), J3.32 (Pin_32)
- new net EPD_DIN: J2.12 (Pin_12), J2.6 (Pin_6), J3.39 (Pin_39), J3.40 (Pin_40)
- new net EPD_RESET: J2.15 (Pin_15), J2.2 (Pin_2), J3.29 (Pin_29), J3.30 (Pin_30)
- new net FRAM_CLK: J3.7 (Pin_7), J3.8 (Pin_8), U1.6 (SCK)
- new net FRAM_CS: J3.13 (Pin_13), J3.14 (Pin_14), U1.1 (CS)
- new net FRAM_RX: J3.11 (Pin_11), J3.12 (Pin_12), U1.2 (SO)
- new net FRAM_TX: J3.10 (Pin_10), J3.9 (Pin_9), U1.5 (SI)
- new net KBD_DEBUG_RX: U2.2 (GPIO1)
- new net KBD_DEBUG_TX: U2.1 (GPIO0)
- new net PERIPHERAL_DEBUG_RX: J3.3 (Pin_3), J3.4 (Pin_4)
- new net PERIPHERAL_DEBUG_TX: J3.1 (Pin_1), J3.2 (Pin_2)
- new net RX: J3.21 (Pin_21), J3.22 (Pin_22), U2.7 (GPIO5)
- new net SD_CLK: J1.5 (CLK), J4.33 (Pin_33), J4.34 (Pin_34)
- new net SD_CS: J1.2 (DAT3/CD), J4.37 (Pin_37), J4.38 (Pin_38)
- new net SD_DET: J4.29 (Pin_29), J4.30 (Pin_30), JP1.1 (A)
- new net SD_RX: J1.7 (DAT0), J4.39 (Pin_39), J4.40 (Pin_40)
- new net SD_TX: J1.3 (CMD), J4.31 (Pin_31), J4.32 (Pin_32)
- new net TX: J3.23 (Pin_23), J3.24 (Pin_24), U2.6 (GPIO4)
- no-connect marks 4 -> 11
Other:
- removed sheet power
- note removed: "16 MHz"
- note removed: "All LEDs SK6805-EC15"
